Commit message: Fixed the incorrect link point for the kinect camera. Implement the home_service robot using rtabmap for the localization.

File: my_robot/urdf/my_robot.xacro (robot description, xacro)
@@ -433,17 +433,10 @@
     <axis xyz="0 1 0" rpy="0 0 0"/>
   </joint>
+  <joint name="camera_optical_joint" type="fixed">
+    <origin xyz="0.075 0 0.125" rpy="-1.5707 0 -1.5707"/>
+    <child link="camera_link_optical"/>
+    <parent link="camera"/>
+  </joint>
   <link name="camera_link_optical">
-    <!--<visual name='camera_visual'>
-      <origin xyz="0 0 0" rpy=" 0 0 0"/>
-      <geometry>
-        <box size="0.05 0.05 0.05"/>
-      </geometry>
-    </visual>-->
-  </link>
-  <joint name="camera_optical_joint" type="fixed">
-    <origin xyz="0.075 0 0.125" rpy="0 0 0"/>
-    <parent link="body"/>
-    <child link="camera_link_optical"/>
-    <axis xyz="0 1 0" rpy="0 0 0"/>
-  </joint>
+  </link>
 </robot>
